File: lumberjack.kicad_pcb (KiCad board)
At the start: 2 copper layers, 284.7 x 94.2 mm, 163 parts, among them J1 USB, J2 AVR_ISP_6, J3 JST, J4 JST, SW1 RESET, SW2 BOOT, U1 ATMEGA328-PU, Y1 16MHz

Commit message: 130423 Update
Finished about 75% of the routing.
Parts:
- MX1, MX10, MX11, MX12, MX13, MX14, MX15, MX16, MX17, MX18, MX19, MX2, MX20, MX21, MX22, MX23, MX24, MX25, MX26, MX27, MX28, MX29, MX3, MX30, MX31, MX32, MX33, MX34, MX35, MX36, MX37, MX38, MX39, MX4, MX40, MX41, MX42, MX43, MX44, MX45, MX46, MX47, MX48, MX49, MX5, MX50, MX51, MX52, MX53, MX54, MX55, MX56, MX57, MX58, MX59, MX6, MX60, MX7, MX9: footprint lumberjack:MX_Alps_Choc -> Library:Lumberjack CherryMX_Choc_v1v2_Hotswap Single Side
- MX8: footprint lumberjack:MX_Alps_Choc_NTHSTH -> Library:Lumberjack CherryMX_Choc_v1v2_Hotswap Single Side
Routing:
- net (no net): track 0.00 -> 672.0 mm, vias 0 -> 2
- net Net-(D62-K): track 231.7 -> 0.00 mm, vias 1 -> 0
- net Net-(D61-K): track 225.7 -> 0.00 mm, vias 1 -> 0
- net Net-(J1-VBUS): track 214.6 -> 0.00 mm
- net Net-(D35-Pad2): track 0.00 -> 160.6 mm
- net Net-(D35-A): track 160.6 -> 0.00 mm
- net Net-(D36-Pad2): track 0.00 -> 134.3 mm
- net Net-(D36-A): track 134.3 -> 0.00 mm
- net Net-(D34-Pad2): track 0.00 -> 129.8 mm
- net Net-(D34-A): track 129.8 -> 0.00 mm
- net Net-(D41-Pad2): track 0.00 -> 95.0 mm
- net Net-(D41-A): track 95.0 -> 0.00 mm
- net Net-(D47-Pad2): track 0.00 -> 75.7 mm
- net Net-(D47-A): track 75.7 -> 0.00 mm
- net Net-(D54-Pad2): track 0.00 -> 64.1 mm
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- removed copper zone on B.Cu, net GND
- removed copper zone on F.Cu, net GND
