File: lumberjack hotswap.kicad_pcb (KiCad board)
At the start: 2 copper layers, 284.7 x 94.2 mm, 163 parts, among them J1 USB, J2 AVR_ISP_6, J3 JST, J4 JST, SW1 RESET, SW2 BOOT, U1 ATMEGA328-PU, Y1 16MHz

Commit message: USB C connector
Updated with USB C connector as a separate board to be soldered on
Parts:
- added ?: , clipboard:7222cb50-ec10-401a-bbd6-f8038f8936cf, F.Cu at (27.3, 61.9)
- added ?: , , F.Cu at (28.9, 66.2)
- added ?: , , F.Cu at (27.4, 50.5)
- added ?: , , F.Cu at (27.3, 66.2)
- added ?: , , F.Cu at (29.0, 50.5)
- J1: moved to F.Cu
- moved J1 16.7 mm to (31.2, 45.2), turned to 180 degrees
- moved H5 4.00 mm to (9.10, 111.3)
- moved H6 4.00 mm to (295.7, 111.3)
Routing:
- net (no net): track 672.0 -> 0.00 mm, vias 2 -> 0
- net Net-(D62-K): track 0.00 -> 241.3 mm, vias 0 -> 1
- net Net-(D61-K): track 0.00 -> 231.5 mm, vias 0 -> 1
- net Net-(J1-VBUS): track 0.00 -> 220.2 mm
- net Net-(D35-A): track 0.00 -> 170.9 mm
- net Net-(D35-Pad2): track 160.6 -> 0.00 mm
- net Net-(D36-A): track 0.00 -> 148.9 mm
- net Net-(D36-Pad2): track 134.3 -> 0.00 mm
- net Net-(D34-A): track 0.00 -> 132.0 mm
- net Net-(D34-Pad2): track 129.8 -> 0.00 mm
- net Net-(D41-A): track 0.00 -> 97.7 mm
- net Net-(D41-Pad2): track 95.0 -> 0.00 mm
- net Net-(D47-A): track 0.00 -> 78.9 mm
- net Net-(D47-Pad2): track 75.7 -> 0.00 mm
- net Net-(D54-A): track 0.00 -> 65.8 mm
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Other:
- board size 284.7 x 94.2 mm -> 284.7 x 109.9 mm
